Commit message: [bee][underactuate] change miniquadrotor urdf

File: robots/mini_quadrotor/urdf/robot.urdf.xacro (robot description, xacro)
@@ -6,7 +6,7 @@
   <thrust_link name="thrust" />
   <!-- kinematics [m] -->
-  <xacro:property name="rotor_x" value="0.085" />
-  <xacro:property name="rotor_y" value="0.085" />
-  <xacro:property name="rotor_z" value="0.026" />
+  <xacro:property name="rotor_x" value="0.1" />
+  <xacro:property name="rotor_y" value="0.1" />
+  <xacro:property name="rotor_z" value="-0.015" />
   <!-- dynamics -->
   <m_f_rate value="-0.011" /> <!-- drag torque rate -->
@@ -96,15 +96,18 @@
   <link name="main_body">
     <inertial>
-      <mass value = "0.832" />
-      <origin xyz="0.002 0 ${0.028 - 0.002}" rpy="0 0 0"/> <!-- TODO: true cog pos -->
+      <origin xyz="-0.00073889 0.00089306 0.01588028" rpy="0 0 0"/>
+      <mass value="1.58195447"/>
       <inertia
-          ixx="0.0030" ixy="0" ixz="0"
-          iyy="0.0030" iyz="0"
-          izz="0.0045"/>
+        ixx="0.00809862"
+        iyy="0.00812972"
+        izz="0.00807423"
+        ixy="0.00002972"
+        ixz="0.00002589"
+        iyz="-0.00003670"/>
     </inertial>
     <visual>
       <origin rpy="0 0 0" xyz="0 0 0"/>
       <geometry>
-        <mesh filename="package://mini_quadrotor/urdf/mesh/main_body_livox.dae" />
+          <mesh filename="package://gimbalrotor/urdf/bee/mesh/full_body_for_underactuate.STL"/>
       </geometry>
     </visual>
@@ -118,5 +121,5 @@
   <!-- spinal -->
   <xacro:extra_module name = "fc" parent = "main_body" visible = "0" >
-    <origin xyz="0 0 0" rpy="0 0 0"/>
+    <origin xyz="-0.0175 0 0.0540" rpy="0 0 0"/>
     <inertial>
       <mass value = "00" />
@@ -137,30 +140,30 @@
     </inertial>
   </xacro:extra_module>
-  <!-- livox mid360 -->
-  <xacro:extra_module name = "lidar_imu" parent = "main_body" visible = "0" > <!-- should be IMU frame -->
-    <origin xyz="${0.011} ${0.02329} ${0.0425 + 0.047 - 0.04412}" rpy="0 0 0"/> <!-- TODO: the true pos -->
-    <inertial>
-      <mass value = "00" />
-      <origin xyz="0 0 0" rpy="0 0 0"/>
-      <inertia
-          ixx="0.0" ixy="0.0" ixz="0.0"
-          iyy="0.0" iyz="0.0" izz="0.0"/>
-    </inertial>
-  </xacro:extra_module>
-  <!-- battery -->
-  <xacro:extra_module name = "battery" parent = "main_body" visible = "1" model_url = "package://mini_quadrotor/urdf/mesh/turnigy_3S_2200mAh.dae" >
-    <origin xyz="0.0 0 -0.035" rpy="${pi/2} 0 0"/>
-    <inertial>
-      <mass value = "0.188" />
-      <origin xyz="0 0 0" rpy="0 0 0"/>
-      <inertia
-          ixx="0.0002" ixy="0.0" ixz="0.0"
-          iyy="0.0002" iyz="0.0" izz="0.0002"/>
-    </inertial>
-  </xacro:extra_module>
+  <!-- <!-\- livox mid360 -\-> -->
+  <!-- <xacro:extra_module name = "lidar_imu" parent = "main_body" visible = "0" > <!-\- should be IMU frame -\-> -->
+  <!--   <origin xyz="${0.011} ${0.02329} ${0.0425 + 0.047 - 0.04412}" rpy="0 0 0"/> <!-\- TODO: the true pos -\-> -->
+  <!--   <inertial> -->
+  <!--     <mass value = "00" /> -->
+  <!--     <origin xyz="0 0 0" rpy="0 0 0"/> -->
+  <!--     <inertia -->
+  <!--         ixx="0.0" ixy="0.0" ixz="0.0" -->
+  <!--         iyy="0.0" iyz="0.0" izz="0.0"/> -->
+  <!--   </inertial> -->
+  <!-- </xacro:extra_module> -->
+  <!-- <!-\- battery -\-> -->
+  <!-- <xacro:extra_module name = "battery" parent = "main_body" visible = "1" model_url = "package://mini_quadrotor/urdf/mesh/turnigy_3S_2200mAh.dae" > -->
+  <!--   <origin xyz="0.0 0 -0.035" rpy="${pi/2} 0 0"/> -->
+  <!--   <inertial> -->
+  <!--     <mass value = "0.188" /> -->
+  <!--     <origin xyz="0 0 0" rpy="0 0 0"/> -->
+  <!--     <inertia -->
+  <!--         ixx="0.0002" ixy="0.0" ixz="0.0" -->
+  <!--         iyy="0.0002" iyz="0.0" izz="0.0002"/> -->
+  <!--   </inertial> -->
+  <!-- </xacro:extra_module> -->
   <!-- propellers -->
-  <xacro:propeller_module id = "1" x = "${-rotor_x}" y = "${-rotor_y}" z = "${rotor_z}" direction = "-1" />
-  <xacro:propeller_module id = "2" x = "${rotor_x}" y = "${-rotor_y}" z = "${rotor_z}" direction = "1" />
-  <xacro:propeller_module id = "3" x = "${rotor_x}" y = "${rotor_y}" z = "${rotor_z}" direction = "-1" />
-  <xacro:propeller_module id = "4" x = "${-rotor_x}" y = "${rotor_y}" z = "${rotor_z}"  direction = "1" />
+  <xacro:propeller_module id = "4" x = "${-rotor_x}" y = "${-rotor_y}" z = "${rotor_z}" direction = "1" />
+  <xacro:propeller_module id = "3" x = "${rotor_x}" y = "${-rotor_y}" z = "${rotor_z}" direction = "-1" />
+  <xacro:propeller_module id = "1" x = "${rotor_x}" y = "${rotor_y}" z = "${rotor_z}" direction = "1" />
+  <xacro:propeller_module id = "2" x = "${-rotor_x}" y = "${rotor_y}" z = "${rotor_z}"  direction = "-1" />
 </robot>
