Commit message: [miniquad][navigation] add movebase navigation and fix param for livox simulation

File: robots/mini_quadrotor/urdf/livox_mid360.gazebo.xacro (robot description, xacro)
@@ -1,5 +1,5 @@
 <?xml version="1.0"?>
 <robot xmlns:xacro="http://www.ros.org/wiki/xacro">
-  <xacro:macro name="livox_mid360_gazebo" params="frame:=lidar_imu tf_prefix:=quadrotor visualize:=True update_rate:=10 resolution:=0.002 noise_mean:=0.0 noise_stddev:=0.01 samples:=24000 downsample:=1 ros_topic:=livox/scan laser_min_range:=0.1 laser_max_range:=200.0">
+  <xacro:macro name="livox_mid360_gazebo" params="frame:=lidar_imu tf_prefix:=quadrotor visualize:=True update_rate:=10 resolution:=0.002 noise_mean:=0.0 noise_stddev:=0.01 samples:=24000 downsample:=1 ros_topic:=livox/lidar_orig laser_min_range:=0.1 laser_max_range:=200.0">
     <gazebo reference="${frame}">
       <sensor type="ray" name="${tf_prefix}/${frame}">
