Commit message: [bee][urdf] modify model inertia

File: robots/gimbalrotor/urdf/bee/gimbalrotor.urdf.xacro (robot description, xacro)
@@ -23,10 +23,16 @@
     <link name="base_link">
       <inertial>
-        <origin xyz="-0.00078520 0.00096010 0.01594366" rpy="0 0 0" />
-        <mass value="1.40419" />
-        <inertia
-            ixx="0.00607504" ixy="0.00014664"  ixz="0.00004521"
-            iyy="0.00609952" iyz="-0.00005926"
-            izz="0.00468030" />
+	<!-- 重心位置 [m]（出力座標系原点→重心） -->
+	<origin xyz="0.00178660 0.00020630 0.01814134" rpy="0 0 0"/>
+	<!-- 質量 [kg] -->
+	<mass value="1.47200040136"/>
+	<!-- 慣性テンソル [kg*m^2]（重心まわり, 正のテンソル表記） -->
+	<inertia
+            ixx="0.00580321693"
+            ixy="0.00006315280"
+            ixz="0.00000697505"
+            iyy="0.00598307897"
+            iyz="-0.00000395631"
+            izz="0.00464383306"/>
       </inertial>
       <visual>

Commit message: [bee][urdf] add livox module in urdf

File: robots/gimbalrotor/urdf/bee/gimbalrotor.urdf.xacro (robot description, xacro)
@@ -229,3 +229,32 @@
     </transmission>
   </xacro:macro>
+  <xacro:macro name="extra_module" params="name parent *origin *inertial visible:=0 model_url:=1 scale:=1">
+    <joint name="${parent}2${name}" type="fixed">
+      <parent link="${parent}"/>
+      <child link="${name}"/>
+      <xacro:insert_block name="origin" />
+    </joint>
+    <link name="${name}">
+      <xacro:insert_block name="inertial" />
+      <xacro:if value="${visible == 1}">
+        <visual>
+          <origin rpy="0 0 0" xyz="0 0 0"/>
+          <geometry>
+            <mesh filename="${model_url}" scale= "${scale} ${scale} ${scale}"/>
+          </geometry>
+        </visual>
+      </xacro:if>
+    </link>
+  </xacro:macro>
+    <!-- livox mid360 -->
+  <xacro:extra_module name = "lidar_imu" parent = "base_link" visible = "0" > <!-- should be IMU frame -->
+    <origin xyz="${0.011} ${0.02329} ${0.072 + 0.047 - 0.04412}" rpy="0 0 0"/> <!-- TODO: the true pos -->
+    <inertial>
+      <mass value = "00" />
+      <origin xyz="0 0 0" rpy="0 0 0"/>
+      <inertia
+          ixx="0.0" ixy="0.0" ixz="0.0"
+          iyy="0.0" iyz="0.0" izz="0.0"/>
+    </inertial>
+  </xacro:extra_module>
 </robot>

Commit message: [bee][urdf] change urdf model with rotorgarde

File: robots/gimbalrotor/urdf/bee/gimbalrotor.urdf.xacro (robot description, xacro)
@@ -138,11 +138,13 @@
     <link name="gimbal_link${self}">
       <inertial>
-        <origin xyz="0.01483947 0.00001426 -0.02606996" rpy="0 0 0"/>
-        <mass value="0.04944"/>
-        <inertia
-            ixx="0.00001165546" ixy="-0.00000000185" ixz="-0.00000168229"
-            iyy="0.00001158109" iyz="-0.00000000588"
-            izz="0.00001018740"
-            />
+        <origin xyz="0.01840184 0.00000854 -0.02830914" rpy="0 0 0" />
+        <mass value="0.08544" />
+        <inertia
+            ixx="0.00009180229"
+            ixy="-0.00000000453"
+            ixz="-0.00000087151"
+            iyy="0.00007733826"
+            iyz="-0.00000000467"
+            izz="0.00014400614" />
       </inertial>
       <collision>
@@ -155,5 +157,5 @@
         <origin xyz="0 0 0" rpy="0 0 0"/>
         <geometry>
-          <mesh filename="package://gimbalrotor/urdf/bee/mesh/rotor_module_downward.STL"/>
+          <mesh filename="package://gimbalrotor/urdf/bee/mesh/rotor_module.STL"/>
         </geometry>
       </visual>

Commit message: [bee][urdf] change direction of battery

File: robots/gimbalrotor/urdf/bee/gimbalrotor.urdf.xacro (robot description, xacro)
@@ -23,16 +23,13 @@
     <link name="base_link">
       <inertial>
-	<!-- 重心位置 [m]（出力座標系原点→重心） -->
-	<origin xyz="0.00178660 0.00020630 0.01814134" rpy="0 0 0"/>
-	<!-- 質量 [kg] -->
-	<mass value="1.47200040136"/>
-	<!-- 慣性テンソル [kg*m^2]（重心まわり, 正のテンソル表記） -->
+	<origin xyz="0.00174386 0.00024903 0.01814134" rpy="0 0 0" />
+	<mass value="1.4720004" />
 	<inertia
-            ixx="0.00580321693"
-            ixy="0.00006315280"
-            ixz="0.00000697505"
-            iyy="0.00598307897"
-            iyz="-0.00000395631"
-            izz="0.00464383306"/>
+            ixx="0.005803188"
+            ixy="0.000063056"
+            ixz="0.000010760"
+            iyy="0.005983301"
+            iyz="-0.000007741"
+            izz="0.004644027" />
       </inertial>
       <visual>

Commit message: [bee][URDF] change position of rotor arm and stl to dae with color and decimate dae

File: robots/gimbalrotor/urdf/bee/gimbalrotor.urdf.xacro (robot description, xacro)
@@ -36,5 +36,5 @@
         <origin xyz="0 0 0" rpy="0 0 0"/>
         <geometry>
-          <mesh filename="package://gimbalrotor/urdf/bee/mesh/base_link.STL"/>
+          <mesh filename="package://gimbalrotor/urdf/bee/mesh/base_link.dae"/>
         </geometry>
       </visual>
@@ -77,5 +77,5 @@
       <parent link="base_link"/>
       <child link="rotor_arm${child1}"/>
-      <origin rpy="0 0 ${pi/4}" xyz="0.036 0.036 0.0165"/>
+      <origin rpy="0 0 ${pi/4}" xyz="0.09035 0.09035 0.0265"/>
       <axis xyz="0 0 1"/>
     </joint>
@@ -93,5 +93,5 @@
       <parent link="base_link"/>
       <child link="rotor_arm${child2}"/>
-      <origin rpy="0 0 ${3*pi/4}" xyz="-0.036 0.036 0.0165"/>
+      <origin rpy="0 0 ${3*pi/4}" xyz="-0.09035 0.09035 0.0265"/>
       <axis xyz="0 0 1"/>
     </joint>
@@ -109,5 +109,5 @@
       <parent link="base_link"/>
       <child link="rotor_arm${child3}"/>
-      <origin rpy="0 0 -${1/4*pi}" xyz="0.036 -0.036 0.0165"/>
+      <origin rpy="0 0 -${1/4*pi}" xyz="0.09035 -0.09035 0.0265"/>
       <axis xyz="0 0 1"/>
     </joint>
@@ -125,5 +125,5 @@
       <parent link="base_link"/>
       <child link="rotor_arm${child4}"/>
-      <origin rpy="0 0 -${3/4*pi}" xyz="-0.036 -0.036 0.0165"/>
+      <origin rpy="0 0 -${3/4*pi}" xyz="-0.09035 -0.09035 0.0265"/>
       <axis xyz="0 0 1"/>
     </joint>
@@ -154,5 +154,5 @@
         <origin xyz="0 0 0" rpy="0 0 0"/>
         <geometry>
-          <mesh filename="package://gimbalrotor/urdf/bee/mesh/rotor_module.STL"/>
+          <mesh filename="package://gimbalrotor/urdf/bee/mesh/rotor_module.dae"/>
         </geometry>
       </visual>
@@ -188,5 +188,5 @@
       <parent link="rotor_arm${self}"/>
       <child link="gimbal_link${self}"/>
-      <origin rpy="0 0 0" xyz="0.077 0 0.0104"/>
+      <origin rpy="0 0 0" xyz="0.0 0 0.0"/>
       <axis xyz="1 0 0"/>
       <dynamics damping="0.8" friction="0.0"/>

Commit message: [bee][urdfconfig] fix rotational limi

File: robots/gimbalrotor/urdf/bee/gimbalrotor.urdf.xacro (robot description, xacro)
@@ -185,5 +185,5 @@
     #### gimbal joints ####
     <joint name="gimbal${self}" type="revolute">
-      <limit effort="6.6" lower="-3.14" upper="3.14" velocity="3.0"/>
+      <limit effort="6.6" lower="-4.5" upper="4.5" velocity="3.0"/>
       <parent link="rotor_arm${self}"/>
       <child link="gimbal_link${self}"/>
