Commit message: [bee_omni] fix urdf stl to dae

File: robots/bee_omni/urdf/bee_omni.urdf.xacro (robot description, xacro)
@@ -17,5 +17,5 @@
         <origin xyz="0 0 0" rpy="0 0 0"/>
         <geometry>
-          <mesh filename="package://gimbalrotor/urdf/bee/mesh/base_link.STL"/>
+          <mesh filename="package://gimbalrotor/urdf/bee/mesh/base_link.dae"/>
         </geometry>
       </visual>
@@ -97,5 +97,5 @@
         <origin xyz="0 0 0" rpy="0 0 0"/>
         <geometry>
-          <mesh filename="package://gimbalrotor/urdf/bee/mesh/rotor_module.STL"/>
+          <mesh filename="package://gimbalrotor/urdf/bee/mesh/rotor_module.dae"/>
         </geometry>
       </visual>

Commit message: [bee_omni][urdf] fix the inertial information of rotor_arm

File: robots/bee_omni/urdf/bee_omni.urdf.xacro (robot description, xacro)
@@ -80,11 +80,13 @@
     <link name="gimbal_link${self}">
       <inertial>
-        <origin xyz="0.01483947 0.00001426 -0.02606996" rpy="0 0 0"/>
-        <mass value="0.04944"/>
-        <inertia
-            ixx="0.00001165546" ixy="-0.00000000185" ixz="-0.00000168229"
-            iyy="0.00001158109" iyz="-0.00000000588"
-            izz="0.00001018740"
-            />
+        <origin xyz="0.01840184 0.00000854 -0.02830914" rpy="0 0 0" />
+        <mass value="0.08544" />
+        <inertia
+            ixx="0.00009180229"
+            ixy="-0.00000000453"
+            ixz="-0.00000087151"
+            iyy="0.00007733826"
+            iyz="-0.00000000467"
+            izz="0.00014400614" />
       </inertial>
       <collision>

Commit message: [bee_omni][urdf][config] remove meanless part of urf and config. and fix counter torque rate.

File: robots/bee_omni/urdf/bee_omni.urdf.xacro (robot description, xacro)
@@ -7,10 +7,13 @@
     <link name="main_body">
       <inertial>
-        <origin xyz="-0.00078520 0.00096010 0.01594366" rpy="0 0 0" />
-        <mass value="1.40419" />
-        <inertia
-            ixx="0.00607504" ixy="0.00014664"  ixz="0.00004521"
-            iyy="0.00609952" iyz="-0.00005926"
-            izz="0.00468030" />
+	<origin xyz="0.00174386 0.00024903 0.01814134" rpy="0 0 0" />
+	<mass value="1.4720004" />
+	<inertia
+            ixx="0.005803188"
+            ixy="0.000063056"
+            ixz="0.000010760"
+            iyy="0.005983301"
+            iyz="-0.000007741"
+            izz="0.004644027" />
       </inertial>
       <visual>
@@ -119,5 +122,5 @@
       <inertial>
         <origin xyz="0 0 0" rpy="0 0 0"/>
-        <mass value="0.005"/>
+        <mass value="0.00001"/>
         <inertia
             ixx="0.001" ixy="0.0" ixz="0.0"
@@ -208,157 +211,3 @@
   <xacro:bee_thrust_link self="3" rotor_direction="-1"/>
   <xacro:bee_thrust_link self="4" rotor_direction="1"/>
-  <!-- <!-\- ============ End‑Effector (EE) =============== -\-> -->
-  <!-- <!-\- Select EE type:  fork | ball | sensor_ball | brush -\-> -->
-  <!-- <xacro:arg name="end_effector" default="fork"/> -->
-  <!-- <xacro:property name="end_effector" value="$(arg end_effector)"/> -->
-  <!-- <!-\- Fixed the flange that all tools attach to -\-> -->
-  <!-- <link name="ee_mount"/> -->
-  <!-- <joint name="body_to_ee_mount" type="fixed"> -->
-  <!--   <parent link="main_body"/> -->
-  <!--   <child link="ee_mount"/> -->
-  <!--   <origin xyz="0 0 0.1725" rpy="0 0 0"/> -->
-  <!-- </joint> -->
-  <!-- <!-\- <!-\\- Tool‑agnostic contact frame (pose set inside each branch) -\\-> -\-> -->
-  <!-- <link name="ee_contact"/> -->
-  <!-- <joint name="ee_mount_to_fork" type="fixed"> -->
-  <!--     <parent link="ee_mount"/> -->
-  <!--     <child link="ee_contact"/> -->
-  <!--     <origin xyz="0 0 0" rpy="0 0 0"/> -->
-  <!-- </joint> -->
-  <!-- <!-\- ############# Fork tool ############# -\-> -->
-  <!-- <xacro:if value="${end_effector == 'fork'}"> -->
-  <!--   <!-\- Tool geometry -\-> -->
-  <!--   <link name="fork"> -->
-  <!--     <inertial> -->
-  <!--       <origin xyz="0.00000000 0.06681059 -0.00005783" rpy="0 0 0"/> -->
-  <!--       <mass value="0.140"/> -->
-  <!--       <inertia -->
-  <!--               ixx="0.00040632" iyy="0.00053824" izz="0.00040617" -->
-  <!--               ixy="0.00000000" ixz="0.00000000" iyz="0.00000000"/> -->
-  <!--     </inertial> -->
-  <!--     <visual> -->
-  <!--       <geometry> -->
-  <!--         <mesh filename="package://beetle_omni/urdf/mesh/end_effector_fork.dae" scale="1 1 1"/> -->
-  <!--       </geometry> -->
-  <!--     </visual> -->
-  <!--   </link> -->
-  <!--   <!-\- Mount fork to the flange -\-> -->
-  <!--   <joint name="ee_mount_to_fork" type="fixed"> -->
-  <!--     <parent link="ee_mount"/> -->
-  <!--     <child link="fork"/> -->
-  <!--     <origin xyz="0 0 0" rpy="0 0 0"/> -->
-  <!--   </joint> -->
-  <!--   <!-\- Contact point for the fork tips -\-> -->
-  <!--   <joint name="fork_to_ee_contact" type="fixed"> -->
-  <!--     <parent link="fork"/> -->
-  <!--     <child link="ee_contact"/> -->
-  <!--     <origin xyz="0 0 0.104" rpy="0 0 0"/> -->
-  <!--   </joint> -->
-  <!-- </xacro:if> -->
-  <!-- <!-\- ############# Ball tool ############# -\-> -->
-  <!-- <xacro:if value="${end_effector == 'ball'}"> -->
-  <!--   <link name="ball"> -->
-  <!--     <inertial> -->
-  <!--       <origin xyz="0.00000000 0.08052689 0.00000000" rpy="0 0 0"/> -->
-  <!--       <mass value="0.1030"/> -->
-  <!--       <inertia -->
-  <!--               ixx="0.00020646" iyy="0.00008167" izz="0.00020646" -->
-  <!--               ixy="0.00000000" ixz="0.00000000" iyz="0.00000000"/> -->
-  <!--     </inertial> -->
-  <!--     <visual> -->
-  <!--       <geometry> -->
-  <!--         <mesh filename="package://beetle_omni/urdf/mesh/end_effector_ball.dae" scale="1 1 1"/> -->
-  <!--       </geometry> -->
-  <!--     </visual> -->
-  <!--   </link> -->
-  <!--   <joint name="ee_mount_to_ball" type="fixed"> -->
-  <!--     <parent link="ee_mount"/> -->
-  <!--     <child link="ball"/> -->
-  <!--     <origin xyz="0 0 0" rpy="0 0 0"/> -->
-  <!--   </joint> -->
-  <!--   <!-\- Contact point at the ball’s center -\-> -->
-  <!--   <joint name="ball_to_ee_contact" type="fixed"> -->
-  <!--     <parent link="ball"/> -->
-  <!--     <child link="ee_contact"/> -->
-  <!--     <origin xyz="0 0 0.11" rpy="0 0 0"/> -->
-  <!--   </joint> -->
-  <!-- </xacro:if> -->
-  <!-- <!-\- ############# Sensor‑ball tool ############# -\-> -->
-  <!-- <xacro:if value="${end_effector == 'sensor_ball'}"> -->
-  <!--   <!-\- Wrench sensor -\-> -->
-  <!--   <link name="wrench_sensor"> -->
-  <!--     <inertial> -->
-  <!--       <origin xyz="0.00000000 0.00000000 -0.01500000" rpy="0 0 0"/> -->
-  <!--       <mass value="0.285"/> -->
-  <!--       <inertia -->
-  <!--               ixx="0.00008773" iyy="0.00012377" izz="0.00016573" -->
-  <!--               ixy="0.00000000" ixz="0.00000328" iyz="0.00000000"/> -->
-  <!--     </inertial> -->
-  <!--     <visual> -->
-  <!--       <geometry> -->
-  <!--         <mesh filename="package://beetle_omni/urdf/mesh/wrench_sensor_pfs055ya501u6.dae" scale="1 1 1"/> -->
-  <!--       </geometry> -->
-  <!--     </visual> -->
-  <!--   </link> -->
-  <!--   <joint name="ee_mount_to_sensor" type="fixed"> -->
-  <!--     <parent link="ee_mount"/> -->
-  <!--     <child link="wrench_sensor"/> -->
-  <!--     <origin xyz="0 0 0.031" rpy="0 0 0"/> -->
-  <!--   </joint> -->
-  <!--   <!-\- Ball attached to the sensor -\-> -->
-  <!--   <link name="ball"> -->
-  <!--     <!-\- (same as plain ball) -\-> -->
-  <!--     <inertial> -->
-  <!--       <origin xyz="0.00000000 0.08052689 0.00000000" rpy="0 0 0"/> -->
-  <!--       <mass value="0.1030"/> -->
-  <!--       <inertia -->
-  <!--               ixx="0.00020646" iyy="0.00008167" izz="0.00020646" -->
-  <!--               ixy="0.00000000" ixz="0.00000000" iyz="0.00000000"/> -->
-  <!--     </inertial> -->
-  <!--     <visual> -->
-  <!--       <geometry> -->
-  <!--         <mesh filename="package://beetle_omni/urdf/mesh/end_effector_ball.dae" scale="1 1 1"/> -->
-  <!--       </geometry> -->
-  <!--     </visual> -->
-  <!--   </link> -->
-  <!--   <joint name="sensor_to_ball" type="fixed"> -->
-  <!--     <parent link="wrench_sensor"/> -->
-  <!--     <child link="ball"/> -->
-  <!--     <origin xyz="0 0 0" rpy="0 0 0"/> -->
-  <!--   </joint> -->
-  <!--   <!-\- Contact point at ball tip -\-> -->
-  <!--   <joint name="ball_to_ee_contact" type="fixed"> -->
-  <!--     <parent link="ball"/> -->
-  <!--     <child link="ee_contact"/> -->
-  <!--     <origin xyz="0 0 0.11" rpy="0 0 0"/> -->
-  <!--   </joint> -->
-  <!-- </xacro:if> -->
-  <!-- <!-\- ############# Brush tool ############# -\-> -->
-  <!-- <xacro:if value="${end_effector == 'brush'}"> -->
-  <!--   <link name="brush"> -->
-  <!--     <inertial> -->
-  <!--       <origin xyz="0.00000000 0.06565796 -0.00001172" rpy="0 0 0"/> -->
-  <!--       <mass value="0.100"/> -->
-  <!--       <inertia -->
-  <!--               ixx="0.00019687" iyy="0.00013173" izz="0.00019689" -->
-  <!--               ixy="0.00000000" ixz="0.00000000" iyz="0.00000000"/> -->
-  <!--     </inertial> -->
-  <!--     <visual> -->
-  <!--       <geometry> -->
-  <!--         <mesh filename="package://beetle_omni/urdf/mesh/end_effector_brush.dae" scale="1 1 1"/> -->
-  <!--       </geometry> -->
-  <!--     </visual> -->
-  <!--   </link> -->
-  <!--   <joint name="ee_mount_to_brush" type="fixed"> -->
-  <!--     <parent link="ee_mount"/> -->
-  <!--     <child link="brush"/> -->
-  <!--     <origin xyz="0 0 0" rpy="0 0 0"/> -->
-  <!--   </joint> -->
-  <!--   <!-\- Contact frame at the bristle tip -\-> -->
-  <!--   <joint name="brush_to_ee_contact" type="fixed"> -->
-  <!--     <parent link="brush"/> -->
-  <!--     <child link="ee_contact"/> -->
-  <!--     <origin xyz="0 0 0.144" rpy="0 0 0"/> -->
-  <!--   </joint> -->
-  <!-- </xacro:if> -->
 </robot>

File: robots/bee_omni/urdf/common.xacro (robot description, xacro)
@@ -1,8 +1,8 @@
 <?xml version="1.0"?>
-<robot xmlns:xacro="http://www.ros.org/wiki/xacro" name="beetle_common" >
+<robot xmlns:xacro="http://www.ros.org/wiki/xacro" name="bee_common" >
   <!-- general attribute -->
   <baselink name="fc" />
   <thrust_link name="thrust" />
-  <m_f_rate value="-0.0165" /> <!-- drag torque rate -->
+  <m_f_rate value="-0.0113" /> <!-- drag torque rate -->
   <xacro:property name="max_force" value="30.0" /> <!-- [N] -->
   <xacro:property name="min_force" value="1.0" /> <!-- [N] -->
