Commit message: [bee] fix build error in bee package

File: robots/bee/urdf/bee.urdf.xacro (robot description, xacro)
@@ -126,4 +126,20 @@
       <child link="rotor_arm${child4}"/>
       <origin rpy="0 0 -${3/4*pi}" xyz="-0.09035 -0.09035 0.0265"/>
+      <axis xyz="0 0 1"/>
+    </joint>
+    <link name="contact_point">
+      <inertial>
+        <origin xyz="0 0 0" rpy="0 0 0"/>
+        <mass value="0.0001"/>
+        <inertia
+            ixx="0.000001" ixy="0.0" ixz="0.0"
+            iyy="0.0001" iyz="0.0"
+            izz="0.0001"/>
+      </inertial>
+    </link>
+    <joint name="cp_base_joint" type="fixed">
+      <parent link="base_link"/>
+      <child link="contact_point"/>
+      <origin rpy="0 0 0" xyz="0.26 0 0"/>
       <axis xyz="0 0 1"/>
     </joint>
