Commit message: [bee][simulation] tune compliant feet and contact solver

File: robots/bee/robots/bee.gazebo.xacro (robot description, xacro)
@@ -10,5 +10,5 @@
   <!-- ODE needs more joint damping than MuJoCo for the same vehicle-level
        settling because the contact solvers regularize impacts differently. -->
-  <xacro:bee_spring_feet stiffness="600.0" damping="20.0"/>
+  <xacro:bee_spring_feet stiffness="1000.0" damping="15.0"/>
   <!-- gazebo plugin for default controller and sensors -->
   <xacro:include filename="$(find aerial_robot_simulation)/xacro/spinal.gazebo.xacro" />

File: robots/bee/urdf/bee_spring_feet.gazebo.xacro (robot description, xacro)
@@ -56,5 +56,5 @@
     </gazebo>
   </xacro:macro>
-  <xacro:macro name="bee_spring_feet" params="stiffness:=600.0 damping:=20.0">
+  <xacro:macro name="bee_spring_feet" params="stiffness:=1000.0 damping:=15.0">
     <material name="bee_spring_shaft_gray">
       <color rgba="0.65 0.65 0.65 1.0"/>
